File: TAPRX-888 KiCad/TAPRX-888.kicad_pcb (KiCad board)
At the start: 6 copper layers, 76 x 100 mm, 222 parts, among them J1 CONN_SMA_JACK_RA, J10 U.FL-R, J11 Conn_JTAG10-mini, J2 CONN_SMA_JACK_RA, J3 CONN_SMA_JACK_RA, J4 CONN_SMA_JACK_RA, J5 USB-3.0, J6 Conn_01x03, J7 Conn_01x03, J8 Conn_01x03, J9 Conn_01x03, Q1 PMOS Si2343DS, Q2 MMBT3904, Q3 PMOS Si2343DS, U1 AP2114H-3.3TRG1, U10 XO-19.2MHZ, U11 CYUSB3014-BZXCT, U14 LP5907MFX-3.3, U16 TLV3501, U18 NC7SV157, U19 74LVC2G14, U2 AP2114H-3.3TRG1, U20 Si5351A, U21 NC7SV157, U22 SN65LVDS1, U3 AP2114H-3.3TRG1, U4 LP5907MFX-3.3, U5 UMW AMS1117-1.2, U6 AD8370, U7 TVS-SP3011, U8 LTC2208CUP_PBF, U9 MX25L3233FM2I, X1 TCXO-27M

Commit message: Added GIT_HASH
per issue #44
Other:
- board text added: "Commit: ${GIT_HASH}"
