File: TAPRX-888 KiCad/Front_End.kicad_sch (KiCad schematic)
At the start: 40 parts, among them J6 Conn_01x03, J7 Conn_01x03, J8 Conn_01x03, J9 Conn_01x03

Commit message: stamp schematic title block with GIT_HASH
Parts:
- U12, U13: value ~ -> (none)
