File: TAPRX-888 KiCad/TAPRX-888.kicad_sch (KiCad schematic)
At the start: 126 parts, among them J1 CONN_SMA_JACK_RA, J11 Conn_JTAG10-mini, J2 CONN_SMA_JACK_RA, J3 CONN_SMA_JACK_RA, J4 CONN_SMA_JACK_RA, J5 USB-3.0, U1 AP2114H-3.3TRG1, U10 XO-19.2MHZ, U11 CYUSB3014-BZXCT, U2 AP2114H-3.3TRG1, U3 AP2114H-3.3TRG1, U4 LP5907MFX-3.3, U5 UMW AMS1117-1.2, U6 AD8370, U7 TVS-SP3011, U8 LTC2208CUP_PBF, U9 MX25L3233FM2I

Commit message: stamp schematic title block with GIT_HASH
Parts:
- H1, H2, H3, H4: value ~ -> (none); now left out of the parts list
