File: TAPRX-888 KiCad/refclk.kicad_sch (KiCad schematic)
At the start: 55 parts, among them J10 U.FL-R, Q1 PMOS Si2343DS, Q2 MMBT3904, Q3 PMOS Si2343DS, U14 LP5907MFX-3.3, U16 TLV3501, U18 NC7SV157, U19 74LVC2G14, U20 Si5351A, U21 NC7SV157, U22 SN65LVDS1, X1 TCXO-27M

Commit message: stamp schematic title block with GIT_HASH
Parts:
- U15, U17: value ~ -> (none)
