File: TAPRX-888.kicad_sch (KiCad schematic)
At the start: 126 parts, among them J1 CONN_SMA_JACK_RA, J11 Conn_JTAG10-mini, J2 CONN_SMA_JACK_RA, J3 CONN_SMA_JACK_RA, J4 CONN_SMA_JACK_RA, J5 USB-3.0, U1 AP2114H-3.3TRG1, U10 XO-19.2MHZ, U11 CYUSB3014-BZXCT, U2 AP2114H-3.3TRG1, U3 AP2114H-3.3TRG1, U4 LP5907MFX-3.3, U5 UMW AMS1117-1.2, U6 AD8370, U7 TVS-SP3011, U8 LTC2208CUP#PBF, U9 MX25L3233FM2I

Commit message: Add title blocks to schematic sheets and PCB
Add a (title_block) to the root/Front_End/refclk schematics and the PCB,
mirroring usb3-fiber's setup: title, date, and rev "DEV". This populates
${TITLE} in the TAPR worksheet frame (the project name was blank before)
and gives ${REVISION} a (rev ...) field for CI provenance injection to
stamp in Phase 2.

Schematic title: "TAPRX-888 HF SDR Receiver"
PCB title:       "TAPRX-888 HF SDR Receiver Board"

Title-block metadata only — no nets, footprints, or geometry changed.

Co-Authored-By: Claude Opus 4.8 <noreply@anthropic.com>
Claude-Session: https://claude.ai/code/session_01TgctKPU2xrNUgrBhHoJD15
Other:
- title: (none) -> TAPRX-888 HF SDR Receiver
Changed lines of the file:
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@@
 	(generator_version "10.0")
 	(paper "A3")
+	(title_block
+		(title "TAPRX-888 HF SDR Receiver")
+		(date "2026-07-16")
+		(rev "DEV")
+	)
 	(text "3.3V"
 		(exclude_from_sim no)
