File: TAPRX-888.kicad_sch (KiCad schematic)
At the start: 126 parts, among them J1 CONN_SMA_JACK_RA, J11 Conn_JTAG10-mini, J2 CONN_SMA_JACK_RA, J3 CONN_SMA_JACK_RA, J4 CONN_SMA_JACK_RA, J5 USB-3.0, U1 AP2114H-3.3TRG1, U10 XO-19.2MHZ, U11 CYUSB3014-BZXCT, U2 AP2114H-3.3TRG1, U3 AP2114H-3.3TRG1, U4 LP5907MFX-3.3, U5 UMW AMS1117-1.2, U6 AD8370, U7 TVS-SP3011, U8 LTC2208CUP#PBF, U9 MX25L3233FM2I

Commit message: Swap in newest design from TAPR/TAPRx888 c01bece; re-graft repo infra
The authoritative HF-SDR design was updated by the hardware designer on
TAPR/TAPRx888 (commit c01bece "proper update", Turn Island Systems). That
branch sits on the pre-flatten layout and also carried a stray
"TAPRX-888 KiCad - Copy/" duplicate + editor lock files, so a plain
cherry-pick was impossible. This lands only the real design edits, mapped
onto ringof's flattened root, and re-applies ringof's infra on top.

Design content taken verbatim from c01bece (mapped to repo root):
  - TAPRX-888.kicad_pcb   (layout/routing/net updates)
  - TAPRX-888.kicad_sch   (root schematic)
  - refclk.kicad_sch      (reference-clock sheet)
  - Library.kicad_sym     (symbol tweak)
  - TAPRX-888.kicad_pro   (used_designators, GIT_HASH text variable)

New file:
  - dru-not-included/TAPRX-888.kicad_dru — USB3 SuperSpeed / USB2 diff-pair
    DRC rules (skew, coupling, via limits, TX-RX isolation). Kept in a
    non-auto-loaded folder to preserve the designer's "not included" intent;
    move to repo root as TAPRX-888.kicad_dru to activate.

Infra re-grafted so nothing ringof added is lost:
  - (title_block) re-added to root/Front_End/refclk schematics + PCB, wired
    to the TAPR.kicad_wks worksheet via page_layout_descr_file in .kicad_pro.
  - Front_End.kicad_sch keeps its title block (designer did not touch it).

Dropped: the committed "Commit: ${GIT_HASH}" silkscreen gr_text on the PCB
(placeholder value; provenance is injected at build time per CLAUDE.md).
The GIT_HASH board property and .kicad_pro text variable remain as the
injection hook.

Co-Authored-By: Claude Opus 4.8 <noreply@anthropic.com>
Claude-Session: https://claude.ai/code/session_019A4jkTeNPLki8CdfTWEUwM
Parts:
- removed J1, J2, J3, J4: CONN_SMA_JACK_RA, TIS_Footprints:SMA-RA-Jack, symbol Library:CONN_SMA_JACK_RA
- added J1, J2, J3, J4: CONN_SMA_JACK_EDGE_JLC_With_Nut, TIS_Footprints:SMA_Jack_EdgeMount_JLC_With_Nut, symbol TIS:CONN_SMA_JACK_EDGE_JLC_with_nut
- H1, H2, H3, H4, TP20: now left out of the parts list
Connections:
- net Clock/EXT_REF_IN: now also J4.1 (In)
- net Front_End_Filter/RF_ATTEN__IN: now also J2.1 (In)
- net Front_End_Filter/RF_IN: now also J1.1 (In)
- net GND: now also J1.2 (Ext), J2.2 (Ext), J3.2 (Ext), J4.2 (Ext)
- net at C27.2, R3.2, R5.1: now also C31.1
- net at C26.2, R2.1, R4.1: now also C30.1
- net at R4.2, U8.8 (AIN+): no longer C30.1
- net at TP1.1: now also J3.1 (In)
- net at R5.2, U8.9 (AIN-): no longer C31.1
Other:
- title: (none) -> TAPRX-888 HF SDR Receiver
- moved on the sheet: C30, C31, R2, R3, R4, R5

Commit message: footprints: put 0603 caps on C_0603; finish schematic TIS liberation
Fixes the one thing that made the board non-reproducible from the library: the
PAD_0603 footprint carried two 3D models (R_0603 for resistors, C_0603 for the
caps placed on it) via a board-level value override a single library footprint
can't express.

PAD_0603 and C_0603 are geometrically identical (same pads/silk), so:
- Reassign the 18 caps on PAD_0603 -> C_0603 (C4,C11-14,C22,C25,C29,C41,C45,C47,
  C51,C52,C57,C60,C62,C65,C78) in both the schematic (Footprint field) and the
  board. Zero copper change. Now PAD_0603 = resistors only (one model), C_0603 =
  caps only (one model); no per-instance model override remains.
- Finish the footprint liberation on the schematic side: re-point every
  schematic Footprint field TIS_Footprints: -> Library: (the board re-point had
  left the schematic mismatched).

Verified: no footprint type has >1 model; schematic Footprint fields == board
footprints for every part; zero TIS references anywhere; parens balanced.

Co-Authored-By: Claude Opus 4.8 <noreply@anthropic.com>
Claude-Session: https://claude.ai/code/session_01A68dcoDnizcNYhKvjGet5a
Parts:
- B1: footprint TIS_Footprints:BUTTON-4p5X4p5 -> Library:BUTTON-4p5X4p5
- C1, C10, C15, C16, C17, C18, C19, C2, C20, C21, C23, C24, C26, C27, C28, C3, C30, C31, C32, C34, C35, C36, C37, C38, C39, C40, C42, C43, C44, C46, C5, C6, C7, C77, C8, C9: footprint TIS_Footprints:C_0603 -> Library:C_0603
- C11, C12, C13, C14, C22, C25, C29, C4, C41, C45, C47: footprint TIS_Footprints:PAD_0603 -> Library:C_0603
- C33: footprint TIS_Footprints:PAD_1206 -> Library:PAD_1206
- D1, D2: footprint TIS_Footprints:SOD-123 -> Library:SOD-123
- D3: footprint TIS_Footprints:LED_RGB_SIDE -> Library:LED_RGB_SIDE
- H1, H2, H3, H4: footprint TIS_Footprints:MountingHole_M2.5-PTH -> Library:MountingHole_M2.5-PTH
- J1, J2, J3, J4: footprint TIS_Footprints:SMA_Jack_EdgeMount_JLC_With_Nut -> Library:SMA_Jack_EdgeMount_JLC_With_Nut
- J11: footprint TIS_Footprints:CONN-JTAG10-mini -> Library:CONN-JTAG10-mini
- J5: footprint TIS_Footprints:USB-3.0 -> Library:USB-3.0
- L1, L3, L4, L5, L6, L7: footprint TIS_Footprints:0603 -> Library:0603
- L2: footprint TIS_Footprints:TIS-Logo -> Library:TIS-Logo
- R1, R13, R14, R15, R16, R17, R18, R19, R2, R20, R21, R22, R23, R24, R25, R26, R27, R3, R4, R5, R58, R59, R6, R7, R8: footprint TIS_Footprints:PAD_0603 -> Library:PAD_0603
- R10, R11, R12, R9: footprint TIS_Footprints:4D02 -> Library:4D02
- TP1, TP10, TP11, TP12, TP13, TP14, TP2, TP3, TP4, TP5, TP6, TP7, TP8, TP9: footprint TIS_Footprints:TP -> Library:TP
- TP20, TP21: footprint TIS_Footprints:TP-Tiny -> Library:TP-Tiny
- U1, U2, U3, U5: footprint TIS_Footprints:SOT-223_THERMAL -> Library:SOT-223_THERMAL
- U10: footprint TIS_Footprints:SMD-2520 -> Library:SMD-2520
- U11: footprint TIS_Footprints:BGA-121 -> Library:BGA-121
- U4: footprint TIS_Footprints:SOT-23-5 -> Library:SOT-23-5
- U6: footprint TIS_Footprints:TSSOP-16-Thermal -> Library:TSSOP-16-Thermal
- U7: footprint TIS_Footprints:SP3011 -> Library:SP3011
- U8: footprint TIS_Footprints:QFN-64_EP_9.5x9.5_Pitch0.5mm -> Library:QFN-64_EP_9.5x9.5_Pitch0.5mm
- U9: footprint TIS_Footprints:SOIC-8-dual -> Library:SOIC-8-dual
- Z1: footprint TIS_Footprints:SOD-323 -> Library:SOD-323

Commit message: symbols: liberate from private TIS/capacitors/resistors libraries
Completes the TIS liberation on the symbol side so every symbol resolves from
the in-repo Library.kicad_sym (the only entry in sym-lib-table):

- Library.kicad_sym: re-point all 71 default Footprint fields TIS_Footprints:
  -> Library:; point the moved 0603 caps' defaults at C_0603 (matching the board).
- Add the 2 symbols that were only cached under foreign nicknames -- C-8.2p-0603
  and CONN_SMA_JACK_EDGE_JLC_with_nut -- into Library.kicad_sym (C-8.2p defaults
  to C_0603).
- Schematics: re-point the foreign symbol lib_ids to Library: -- TIS: (SMA J1-J4,
  4), capacitors: (C78, 1), resistors: (R-100-0603, 1) -- updating instances and
  lib_symbols cache keys. R-100-0603 already had a Library: cache, so its orphaned
  resistors: cache entry was removed rather than duplicated.

Verified: only the Library nickname remains; 75/75 schematic symbols resolve in
Library.kicad_sym; zero TIS references in symbols/schematics/board; no duplicate
cache keys; every instance resolves; schematic Footprint == board; parens balanced.

Co-Authored-By: Claude Opus 4.8 <noreply@anthropic.com>
Claude-Session: https://claude.ai/code/session_01A68dcoDnizcNYhKvjGet5a
Parts:
- J1, J2, J3, J4: symbol TIS:CONN_SMA_JACK_EDGE_JLC_with_nut -> Library:CONN_SMA_JACK_EDGE_JLC_with_nut
Changed lines of the file:
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@@
 	)
 	(symbol
-		(lib_id "TIS:CONN_SMA_JACK_EDGE_JLC_with_nut")
+		(lib_id "Library:CONN_SMA_JACK_EDGE_JLC_with_nut")
 		(at 25.4 62.23 0)
 		(mirror y)
@@
 	)
 	(symbol
-		(lib_id "TIS:CONN_SMA_JACK_EDGE_JLC_with_nut")
+		(lib_id "Library:CONN_SMA_JACK_EDGE_JLC_with_nut")
 		(at 25.4 41.91 0)
 		(mirror y)
@@
 	)
 	(symbol
-		(lib_id "TIS:CONN_SMA_JACK_EDGE_JLC_with_nut")
+		(lib_id "Library:CONN_SMA_JACK_EDGE_JLC_with_nut")
 		(at 22.86 125.73 0)
 		(mirror y)
@@
 	)
 	(symbol
-		(lib_id "TIS:CONN_SMA_JACK_EDGE_JLC_with_nut")
+		(lib_id "Library:CONN_SMA_JACK_EDGE_JLC_with_nut")
 		(at 25.4 21.59 0)
 		(mirror y)
