File: TAPRX-888.kicad_sch (KiCad schematic)
At the start: 126 parts, among them J1 CONN_SMA_JACK_EDGE_JLC_With_N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, J11 Conn_JTAG10-mini, J2 CONN_SMA_JACK_EDGE_JLC_With_N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, J3 CONN_SMA_JACK_EDGE_JLC_With_N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, J4 CONN_SMA_JACK_EDGE_JLC_With_N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, J5 USB-3.0, U1 AP2114H-3.3TRG1, U10 XO-19.2MHZ, U11 CYUSB3014-BZXCT, U2 AP2114H-3.3TRG1, U3 AP2114H-3.3TRG1, U4 LP5907MFX-3.3, U5 UMW AMS1117-1.2, U6 AD8370, U7 TVS-SP3011, U8 LTC2208CUP#PBF, U9 MX25L3233FM2I

Commit message: DNP the testpoints for 3D model clarity
Parts:
- TP1, TP10, TP11, TP12, TP13, TP14, TP2, TP20, TP3, TP4, TP5, TP6, TP7, TP8, TP9: now not fitted
- TP21: now not fitted; now left out of the parts list
Changed lines of the file:
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@@
 		(in_bom no)
 		(on_board yes)
-		(in_pos_files no)
-		(dnp no)
+		(in_pos_files yes)
+		(dnp yes)
 		(property "Reference" "TP20"
 			(at 267.462 190.5 0)
@@
 		(on_board yes)
 		(in_pos_files yes)
-		(dnp no)
+		(dnp yes)
 		(property "Reference" "TP10"
 			(at 198.12 16.51 0)
@@
 		(body_style 1)
 		(exclude_from_sim no)
-		(in_bom yes)
+		(in_bom no)
 		(on_board yes)
 		(in_pos_files yes)
-		(dnp no)
+		(dnp yes)
 		(property "Reference" "TP21"
 			(at 269.24 193.0399 0)
@@
 		(on_board yes)
 		(in_pos_files yes)
-		(dnp no)
+		(dnp yes)
 		(fields_autoplaced yes)
 		(property "Reference" "TP6"
@@
 		(on_board yes)
 		(in_pos_files yes)
-		(dnp no)
+		(dnp yes)
 		(property "Reference" "TP13"
 			(at 389.89 226.0599 0)
@@
 		(on_board yes)
 		(in_pos_files yes)
-		(dnp no)
+		(dnp yes)
 		(fields_autoplaced yes)
 		(property "Reference" "TP4"
@@
 		(on_board yes)
 		(in_pos_files yes)
-		(dnp no)
+		(dnp yes)
 		(fields_autoplaced yes)
 		(property "Reference" "TP2"
@@
 		(on_board yes)
 		(in_pos_files yes)
-		(dnp no)
+		(dnp yes)
 		(property "Reference" "TP11"
 			(at 271.78 114.2999 0)
@@
 		(on_board yes)
 		(in_pos_files yes)
-		(dnp no)
+		(dnp yes)
 		(fields_autoplaced yes)
 		(property "Reference" "TP7"
@@
 		(on_board yes)
 		(in_pos_files yes)
-		(dnp no)
+		(dnp yes)
 		(fields_autoplaced yes)
 		(property "Reference" "TP1"
@@
 		(in_bom no)
 		(on_board yes)
-		(in_pos_files no)
-		(dnp no)
+		(in_pos_files yes)
+		(dnp yes)
 		(property "Reference" "TP14"
 			(at 397.51 242.5699 0)
@@
 		(on_board yes)
 		(in_pos_files yes)
-		(dnp no)
+		(dnp yes)
 		(fields_autoplaced yes)
 		(property "Reference" "TP5"
@@
 		(on_board yes)
 		(in_pos_files yes)
-		(dnp no)
+		(dnp yes)
 		(fields_autoplaced yes)
 		(property "Reference" "TP8"
@@
 		(on_board yes)
 		(in_pos_files yes)
-		(dnp no)
+		(dnp yes)
 		(property "Reference" "TP12"
 			(at 271.78 116.8399 0)
@@
 		(on_board yes)
 		(in_pos_files yes)
-		(dnp no)
+		(dnp yes)
 		(property "Reference" "TP3"
 			(at 89.1032 99.568 0)
@@
 		(on_board yes)
 		(in_pos_files yes)
-		(dnp no)
+		(dnp yes)
 		(property "Reference" "TP9"
 			(at 198.628 19.304 0)
