File: refclk.kicad_sch (KiCad schematic)
At the start: 55 parts, among them J10 U.FL-R, Q1 PMOS Si2343DS, Q2 MMBT3904, Q3 PMOS Si2343DS, U14 LP5907MFX-3.3, U16 TLV3501, U18 NC7SV157, U19 74LVC2G14, U20 Si5351A, U21 NC7SV157, U22 SN65LVDS1, X1 TCXO-27M

Commit message: Add title blocks to schematic sheets and PCB
Add a (title_block) to the root/Front_End/refclk schematics and the PCB,
mirroring usb3-fiber's setup: title, date, and rev "DEV". This populates
${TITLE} in the TAPR worksheet frame (the project name was blank before)
and gives ${REVISION} a (rev ...) field for CI provenance injection to
stamp in Phase 2.

Schematic title: "TAPRX-888 HF SDR Receiver"
PCB title:       "TAPRX-888 HF SDR Receiver Board"

Title-block metadata only — no nets, footprints, or geometry changed.

Co-Authored-By: Claude Opus 4.8 <noreply@anthropic.com>
Claude-Session: https://claude.ai/code/session_01TgctKPU2xrNUgrBhHoJD15
Other:
- title: (none) -> TAPRX-888 HF SDR Receiver
Changed lines of the file:
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@@
 	(generator_version "10.0")
 	(paper "A4")
+	(title_block
+		(title "TAPRX-888 HF SDR Receiver")
+		(date "2026-07-16")
+		(rev "DEV")
+	)
 	(junction
 		(at 266.7 50.8)
