File: refclk.kicad_sch (KiCad schematic)
At the start: 55 parts, among them J10 U.FL-R, Q1 PMOS Si2343DS, Q2 MMBT3904, Q3 PMOS Si2343DS, U14 LP5907MFX-3.3, U16 TLV3501, U18 NC7SV157, U19 74LVC2G14, U20 Si5351A, U21 NC7SV157, U22 SN65LVDS1, X1 TCXO-27M

Commit message: Swap in newest design from TAPR/TAPRx888 c01bece; re-graft repo infra
The authoritative HF-SDR design was updated by the hardware designer on
TAPR/TAPRx888 (commit c01bece "proper update", Turn Island Systems). That
branch sits on the pre-flatten layout and also carried a stray
"TAPRX-888 KiCad - Copy/" duplicate + editor lock files, so a plain
cherry-pick was impossible. This lands only the real design edits, mapped
onto ringof's flattened root, and re-applies ringof's infra on top.

Design content taken verbatim from c01bece (mapped to repo root):
  - TAPRX-888.kicad_pcb   (layout/routing/net updates)
  - TAPRX-888.kicad_sch   (root schematic)
  - refclk.kicad_sch      (reference-clock sheet)
  - Library.kicad_sym     (symbol tweak)
  - TAPRX-888.kicad_pro   (used_designators, GIT_HASH text variable)

New file:
  - dru-not-included/TAPRX-888.kicad_dru — USB3 SuperSpeed / USB2 diff-pair
    DRC rules (skew, coupling, via limits, TX-RX isolation). Kept in a
    non-auto-loaded folder to preserve the designer's "not included" intent;
    move to repo root as TAPRX-888.kicad_dru to activate.

Infra re-grafted so nothing ringof added is lost:
  - (title_block) re-added to root/Front_End/refclk schematics + PCB, wired
    to the TAPR.kicad_wks worksheet via page_layout_descr_file in .kicad_pro.
  - Front_End.kicad_sch keeps its title block (designer did not touch it).

Dropped: the committed "Commit: ${GIT_HASH}" silkscreen gr_text on the PCB
(placeholder value; provenance is injected at build time per CLAUDE.md).
The GIT_HASH board property and .kicad_pro text variable remain as the
injection hook.

Co-Authored-By: Claude Opus 4.8 <noreply@anthropic.com>
Claude-Session: https://claude.ai/code/session_019A4jkTeNPLki8CdfTWEUwM
Parts:
- added C78: C-8.2p-0603, TIS_Footprints:PAD_0603, symbol capacitors:C-8.2p-0603
- added R61: R-100-0603, TIS_Footprints:PAD_0603, symbol resistors:R-100-0603
Connections:
- net SCLKN: now also C78.2, R61.2
- net SCLKP: now also C78.1, R61.1
Other:
- title: (none) -> TAPRX-888 HF SDR Receiver
- moved on the sheet: C76, J10, R56, U22

Commit message: footprints: put 0603 caps on C_0603; finish schematic TIS liberation
Fixes the one thing that made the board non-reproducible from the library: the
PAD_0603 footprint carried two 3D models (R_0603 for resistors, C_0603 for the
caps placed on it) via a board-level value override a single library footprint
can't express.

PAD_0603 and C_0603 are geometrically identical (same pads/silk), so:
- Reassign the 18 caps on PAD_0603 -> C_0603 (C4,C11-14,C22,C25,C29,C41,C45,C47,
  C51,C52,C57,C60,C62,C65,C78) in both the schematic (Footprint field) and the
  board. Zero copper change. Now PAD_0603 = resistors only (one model), C_0603 =
  caps only (one model); no per-instance model override remains.
- Finish the footprint liberation on the schematic side: re-point every
  schematic Footprint field TIS_Footprints: -> Library: (the board re-point had
  left the schematic mismatched).

Verified: no footprint type has >1 model; schematic Footprint fields == board
footprints for every part; zero TIS references anywhere; parens balanced.

Co-Authored-By: Claude Opus 4.8 <noreply@anthropic.com>
Claude-Session: https://claude.ai/code/session_01A68dcoDnizcNYhKvjGet5a
Parts:
- C62, C65, C78: footprint TIS_Footprints:PAD_0603 -> Library:C_0603
- C63, C64, C66, C67, C68, C69, C70, C71, C72, C73, C74, C75, C76: footprint TIS_Footprints:C_0603 -> Library:C_0603
- J10: footprint TIS_Footprints:HRS_U.FL-R-SMT(01) -> Library:HRS_U.FL-R-SMT(01)
- L15, L16, L17: footprint TIS_Footprints:0603 -> Library:0603
- Q1, Q2, Q3, U15, U17: footprint TIS_Footprints:SOT-23 -> Library:SOT-23
- R41, R42, R43, R44, R45, R46, R47, R48, R49, R50, R51, R52, R53, R54, R55, R56, R57, R60, R61: footprint TIS_Footprints:PAD_0603 -> Library:PAD_0603
- TP15, TP16, TP17, TP18, TP19: footprint TIS_Footprints:TP -> Library:TP
- U14, U22: footprint TIS_Footprints:SOT-23-5 -> Library:SOT-23-5
- U16: footprint TIS_Footprints:SOT-23-6 -> Library:SOT-23-6
- U18, U21: footprint TIS_Footprints:SC-70-6 -> Library:SC-70-6
- U19: footprint TIS_Footprints:SC-70-6_rot90 -> Library:SC-70-6_rot90
- U20: footprint TIS_Footprints:MSOP-10_W3mm -> Library:MSOP-10_W3mm
- X1: footprint TIS_Footprints:TCXO-3225 -> Library:TCXO-3225
Changed lines of the file:
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@@
 			)
 		)
-		(property "Footprint" "TIS_Footprints:SOT-23"
+		(property "Footprint" "Library:SOT-23"
 			(at 109.855 34.29 0)
 			(hide yes)
@@
 			)
 		)
-		(property "Footprint" "TIS_Footprints:SOT-23-6"
+		(property "Footprint" "Library:SOT-23-6"
 			(at 111.76 88.9 0)
 			(hide yes)
@@
 			)
 		)
-		(property "Footprint" "TIS_Footprints:TP"
+		(property "Footprint" "Library:TP"
 			(at 85.09 161.29 0)
 			(hide yes)
@@
 			)
 		)
-		(property "Footprint" "TIS_Footprints:C_0603"
+		(property "Footprint" "Library:C_0603"
 			(at 138.176 39.878 0)
 			(hide yes)
@@
 			)
 		)
-		(property "Footprint" "TIS_Footprints:SOT-23-5"
+		(property "Footprint" "Library:SOT-23-5"
 			(at 234.95 52.07 0)
 			(hide yes)
@@
 			)
 		)
-		(property "Footprint" "TIS_Footprints:HRS_U.FL-R-SMT(01)"
+		(property "Footprint" "Library:HRS_U.FL-R-SMT(01)"
 			(at 219.71 10.16 0)
 			(hide yes)
@@
 			)
 		)
-		(property "Footprint" "TIS_Footprints:TCXO-3225"
+		(property "Footprint" "Library:TCXO-3225"
 			(at 153.67 58.42 0)
 			(hide yes)
@@
 			)
 		)
-		(property "Footprint" "TIS_Footprints:0603"
+		(property "Footprint" "Library:0603"
 			(at 128.778 27.178 0)
 			(hide yes)
@@
 			)
 		)
-		(property "Footprint" "TIS_Footprints:PAD_0603"
+		(property "Footprint" "Library:PAD_0603"
 			(at 173.736 120.904 90)
 			(hide yes)
@@
 			)
 		)
-		(property "Footprint" "TIS_Footprints:C_0603"
+		(property "Footprint" "Library:C_0603"
 			(at 189.484 79.502 0)
 			(hide yes)
@@
 			)
 		)
-		(property "Footprint" "TIS_Footprints:C_0603"
+		(property "Footprint" "Library:C_0603"
 			(at 205.994 141.732 0)
 			(hide yes)
@@
 			)
 		)
-		(property "Footprint" "TIS_Footprints:PAD_0603"
+		(property "Footprint" "Library:PAD_0603"
 			(at 247.396 29.464 90)
 			(hide yes)
@@
 			)
 		)
-		(property "Footprint" "TIS_Footprints:SOT-23"
+		(property "Footprint" "Library:SOT-23"
 			(at 58.928 123.317 0)
 			(hide yes)
@@
 			)
 		)
-		(property "Footprint" "TIS_Footprints:C_0603"
+		(property "Footprint" "Library:C_0603"
 			(at 232.156 112.268 0)
 			(hide yes)
@@
 			)
 		)
-		(property "Footprint" "TIS_Footprints:C_0603"
+		(property "Footprint" "Library:C_0603"
 			(at 241.554 49.022 0)
 			(hide yes)
@@
 			)
 		)
-		(property "Footprint" "TIS_Footprints:SOT-23"
+		(property "Footprint" "Library:SOT-23"
 			(at 132.588 141.097 0)
 			(hide yes)
@@
 			)
 		)
-		(property "Footprint" "TIS_Footprints:PAD_0603"
+		(property "Footprint" "Library:PAD_0603"
 			(at 218.186 90.424 90)
 			(hide yes)
@@
 			)
 		)
-		(property "Footprint" "TIS_Footprints:PAD_0603"
+		(property "Footprint" "Library:PAD_0603"
 			(at 232.156 156.464 90)
 			(hide yes)
@@
 			)
 		)
-		(property "Footprint" "TIS_Footprints:C_0603"
+		(property "Footprint" "Library:C_0603"
 			(at 254.254 144.272 0)
 			(hide yes)
@@
 			)
 		)
-		(property "Footprint" "TIS_Footprints:TP"
+		(property "Footprint" "Library:TP"
 			(at 26.67 100.33 0)
 			(hide yes)
@@
 			)
 		)
-		(property "Footprint" "TIS_Footprints:0603"
+		(property "Footprint" "Library:0603"
 			(at 222.758 99.568 0)
 			(hide yes)
@@
 			)
 		)
-		(property "Footprint" "TIS_Footprints:C_0603"
+		(property "Footprint" "Library:C_0603"
 			(at 131.318 131.064 0)
 			(hide yes)
@@
 			)
 		)
-		(property "Footprint" "TIS_Footprints:0603"
+		(property "Footprint" "Library:0603"
 			(at 44.958 46.228 0)
 			(hide yes)
@@
 			)
 		)
-		(property "Footprint" "TIS_Footprints:TP"
+		(property "Footprint" "Library:TP"
 			(at 26.67 104.14 0)
 			(hide yes)
@@
 			)
 		)
-		(property "Footprint" "TIS_Footprints:SC-70-6"
+		(property "Footprint" "Library:SC-70-6"
 			(at 240.03 148.59 0)
 			(hide yes)
@@
 			)
 		)
-		(property "Footprint" "TIS_Footprints:PAD_0603"
+		(property "Footprint" "Library:PAD_0603"
 			(at 79.756 76.454 90)
 			(hide yes)
@@
 			)
 		)
-		(property "Footprint" "TIS_Footprints:PAD_0603"
+		(property "Footprint" "Library:PAD_0603"
 			(at 152.146 139.954 90)
 			(hide yes)
@@
 			)
 		)
-		(property "Footprint" "TIS_Footprints:SC-70-6"
+		(property "Footprint" "Library:SC-70-6"
 			(at 177.8 78.74 0)
 			(hide yes)
@@
 			)
 		)
-		(property "Footprint" "TIS_Footprints:PAD_0603"
+		(property "Footprint" "Library:PAD_0603"
 			(at 79.756 61.214 90)
 			(hide yes)
@@
 			)
 		)
-		(property "Footprint" "TIS_Footprints:PAD_0603"
+		(property "Footprint" "Library:PAD_0603"
 			(at 251.206 61.214 90)
 			(hide yes)
@@
 			)
 		)
-		(property "Footprint" "TIS_Footprints:PAD_0603"
+		(property "Footprint" "Library:PAD_0603"
 			(at 38.354 155.194 90)
 			(hide yes)
@@
 			)
 		)
-		(property "Footprint" "TIS_Footprints:TP"
+		(property "Footprint" "Library:TP"
 			(at 128.27 104.14 0)
 			(hide yes)
@@
 			)
 		)
-		(property "Footprint" "TIS_Footprints:SOT-23-5"
+		(property "Footprint" "Library:SOT-23-5"
 			(at 53.34 165.1 0)
 			(hide yes)
@@
 			)
 		)
-		(property "Footprint" "TIS_Footprints:PAD_0603"
+		(property "Footprint" "Library:PAD_0603"
 			(at 45.466 106.934 90)
 			(hide yes)
@@
 			)
 		)
-		(property "Footprint" "TIS_Footprints:PAD_0603"
+		(property "Footprint" "Library:PAD_0603"
 			(at 158.496 134.366 90)
 			(hide yes)
@@
 			)
 		)
-		(property "Footprint" "TIS_Footprints:SC-70-6_rot90"
+		(property "Footprint" "Library:SC-70-6_rot90"
 			(at 198.12 140.97 0)
 			(hide yes)
@@
 			)
 		)
-		(property "Footprint" "TIS_Footprints:PAD_0603"
+		(property "Footprint" "Library:PAD_0603"
 			(at 64.516 80.264 90)
 			(hide yes)
@@
 			)
 		)
-		(property "Footprint" "TIS_Footprints:PAD_0603"
+		(property "Footprint" "Library:PAD_0603"
 			(at 228.346 25.654 90)
 			(hide yes)
@@
 			)
 		)
-		(property "Footprint" "TIS_Footprints:C_0603"
+		(property "Footprint" "Library:C_0603"
 			(at 54.356 58.928 0)
 			(hide yes)
@@
 			)
 		)
-		(property "Footprint" "TIS_Footprints:PAD_0603"
+		(property "Footprint" "Library:C_0603"
 			(at 68.834 174.752 0)
 			(hide yes)
@@
 			)
 		)
-		(property "Footprint" "TIS_Footprints:C_0603"
+		(property "Footprint" "Library:C_0603"
 			(at 85.344 73.152 0)
 			(hide yes)
@@
 			)
 		)
-		(property "Footprint" "TIS_Footprints:PAD_0603"
+		(property "Footprint" "Library:PAD_0603"
 			(at 88.646 102.616 90)
 			(hide yes)
@@
 			)
 		)
-		(property "Footprint" "TIS_Footprints:PAD_0603"
+		(property "Footprint" "Library:C_0603"
 			(at 265.684 20.574 0)
 			(hide yes)
@@
 			)
 		)
-		(property "Footprint" "TIS_Footprints:C_0603"
+		(property "Footprint" "Library:C_0603"
 			(at 92.964 112.522 0)
 			(hide yes)
@@
 			)
 		)
-		(property "Footprint" "TIS_Footprints:PAD_0603"
+		(property "Footprint" "Library:PAD_0603"
 			(at 64.516 37.084 90)
 			(hide yes)
@@
 			)
 		)
-		(property "Footprint" "TIS_Footprints:SOT-23"
+		(property "Footprint" "Library:SOT-23"
 			(at 64.135 19.05 0)
 			(hide yes)
@@
 			)
 		)
-		(property "Footprint" "TIS_Footprints:PAD_0603"
+		(property "Footprint" "Library:PAD_0603"
 			(at 40.386 106.934 90)
 			(hide yes)
@@
 			)
 		)
-		(property "Footprint" "TIS_Footprints:C_0603"
+		(property "Footprint" "Library:C_0603"
 			(at 53.848 99.314 0)
 			(hide yes)
@@
 			)
 		)
-		(property "Footprint" "TIS_Footprints:PAD_0603"
+		(property "Footprint" "Library:PAD_0603"
 			(at 73.406 102.616 90)
 			(hide yes)
@@
 			)
 		)
-		(property "Footprint" "TIS_Footprints:SOT-23"
+		(property "Footprint" "Library:SOT-23"
 			(at 175.26 135.255 0)
 			(hide yes)
@@
 			)
 		)
-		(property "Footprint" "TIS_Footprints:TP"
+		(property "Footprint" "Library:TP"
 			(at 128.27 100.33 0)
 			(hide yes)
@@
 			)
 		)
-		(property "Footprint" "TIS_Footprints:PAD_0603"
+		(property "Footprint" "Library:PAD_0603"
 			(at 96.266 86.614 90)
 			(hide yes)
@@
 			)
 		)
-		(property "Footprint" "TIS_Footprints:C_0603"
+		(property "Footprint" "Library:C_0603"
 			(at 181.864 145.542 0)
 			(hide yes)
@@
 			)
 		)
-		(property "Footprint" "TIS_Footprints:PAD_0603"
+		(property "Footprint" "Library:PAD_0603"
 			(at 211.836 90.424 90)
 			(hide yes)
@@
 			)
 		)
-		(property "Footprint" "TIS_Footprints:MSOP-10_W3mm"
+		(property "Footprint" "Library:MSOP-10_W3mm"
 			(at 231.14 85.09 0)
 			(hide yes)
@@
 			)
 		)
-		(property "Footprint" "TIS_Footprints:PAD_0603"
+		(property "Footprint" "Library:C_0603"
 			(at 46.736 171.704 0)
 			(hide yes)
@@
 			)
 		)
-		(property "Footprint" "TIS_Footprints:C_0603"
+		(property "Footprint" "Library:C_0603"
 			(at 246.126 112.268 0)
 			(hide yes)

Commit message: symbols: liberate from private TIS/capacitors/resistors libraries
Completes the TIS liberation on the symbol side so every symbol resolves from
the in-repo Library.kicad_sym (the only entry in sym-lib-table):

- Library.kicad_sym: re-point all 71 default Footprint fields TIS_Footprints:
  -> Library:; point the moved 0603 caps' defaults at C_0603 (matching the board).
- Add the 2 symbols that were only cached under foreign nicknames -- C-8.2p-0603
  and CONN_SMA_JACK_EDGE_JLC_with_nut -- into Library.kicad_sym (C-8.2p defaults
  to C_0603).
- Schematics: re-point the foreign symbol lib_ids to Library: -- TIS: (SMA J1-J4,
  4), capacitors: (C78, 1), resistors: (R-100-0603, 1) -- updating instances and
  lib_symbols cache keys. R-100-0603 already had a Library: cache, so its orphaned
  resistors: cache entry was removed rather than duplicated.

Verified: only the Library nickname remains; 75/75 schematic symbols resolve in
Library.kicad_sym; zero TIS references in symbols/schematics/board; no duplicate
cache keys; every instance resolves; schematic Footprint == board; parens balanced.

Co-Authored-By: Claude Opus 4.8 <noreply@anthropic.com>
Claude-Session: https://claude.ai/code/session_01A68dcoDnizcNYhKvjGet5a
Parts:
- C78: symbol capacitors:C-8.2p-0603 -> Library:C-8.2p-0603
- R61: symbol resistors:R-100-0603 -> Library:R-100-0603
Changed lines of the file:
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@@
 	)
 	(symbol
-		(lib_id "resistors:R-100-0603")
+		(lib_id "Library:R-100-0603")
 		(at 246.38 29.21 0)
 		(unit 1)
@@
 	)
 	(symbol
-		(lib_id "capacitors:C-8.2p-0603")
+		(lib_id "Library:C-8.2p-0603")
 		(at 266.7 29.21 0)
 		(unit 1)
