File: refclk.kicad_sch (KiCad schematic)
At the start: 57 parts, among them J10 U.FL-R, Q1 PMOS Si2343DS, Q2 MMBT3904, Q3 PMOS Si2343DS, U14 LP5907MFX-3.3, U16 TLV3501, U18 NC7SV157, U19 74LVC2G14, U20 Si5351A, U21 NC7SV157, U22 SN65LVDS1, X1 TCXO-27M

Commit message: DNP the testpoints for 3D model clarity
Parts:
- TP15, TP16, TP17, TP18, TP19: now not fitted
Changed lines of the file:
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@@
 		(on_board yes)
 		(in_pos_files yes)
-		(dnp no)
+		(dnp yes)
 		(property "Reference" "TP17"
 			(at 90.3732 168.148 0)
@@
 		(on_board yes)
 		(in_pos_files yes)
-		(dnp no)
+		(dnp yes)
 		(property "Reference" "TP15"
 			(at 29.718 106.426 0)
@@
 		(on_board yes)
 		(in_pos_files yes)
-		(dnp no)
+		(dnp yes)
 		(property "Reference" "TP16"
 			(at 29.718 110.998 0)
@@
 		(on_board yes)
 		(in_pos_files yes)
-		(dnp no)
+		(dnp yes)
 		(property "Reference" "TP19"
 			(at 133.5532 110.998 0)
@@
 		(on_board yes)
 		(in_pos_files yes)
-		(dnp no)
+		(dnp yes)
 		(property "Reference" "TP18"
 			(at 133.5532 107.188 0)
