File: Front_End.kicad_sch (KiCad schematic)
At the start: 40 parts, among them J6 Conn_01x03, J7 Conn_01x03, J8 Conn_01x03, J9 Conn_01x03

Commit message: Swap in newest design from TAPR/TAPRx888 c01bece; re-graft repo infra
The authoritative HF-SDR design was updated by the hardware designer on
TAPR/TAPRx888 (commit c01bece "proper update", Turn Island Systems). That
branch sits on the pre-flatten layout and also carried a stray
"TAPRX-888 KiCad - Copy/" duplicate + editor lock files, so a plain
cherry-pick was impossible. This lands only the real design edits, mapped
onto ringof's flattened root, and re-applies ringof's infra on top.

Design content taken verbatim from c01bece (mapped to repo root):
  - TAPRX-888.kicad_pcb   (layout/routing/net updates)
  - TAPRX-888.kicad_sch   (root schematic)
  - refclk.kicad_sch      (reference-clock sheet)
  - Library.kicad_sym     (symbol tweak)
  - TAPRX-888.kicad_pro   (used_designators, GIT_HASH text variable)

New file:
  - dru-not-included/TAPRX-888.kicad_dru — USB3 SuperSpeed / USB2 diff-pair
    DRC rules (skew, coupling, via limits, TX-RX isolation). Kept in a
    non-auto-loaded folder to preserve the designer's "not included" intent;
    move to repo root as TAPRX-888.kicad_dru to activate.

Infra re-grafted so nothing ringof added is lost:
  - (title_block) re-added to root/Front_End/refclk schematics + PCB, wired
    to the TAPR.kicad_wks worksheet via page_layout_descr_file in .kicad_pro.
  - Front_End.kicad_sch keeps its title block (designer did not touch it).

Dropped: the committed "Commit: ${GIT_HASH}" silkscreen gr_text on the PCB
(placeholder value; provenance is injected at build time per CLAUDE.md).
The GIT_HASH board property and .kicad_pro text variable remain as the
injection hook.

Co-Authored-By: Claude Opus 4.8 <noreply@anthropic.com>
Claude-Session: https://claude.ai/code/session_019A4jkTeNPLki8CdfTWEUwM
Other:
- title: (none) -> TAPRX-888 HF SDR Receiver
Changed lines of the file:
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@@
 	(generator_version "10.0")
 	(paper "A4")
+	(title_block
+		(title "TAPRX-888 HF SDR Receiver")
+		(date "2026-07-16")
+		(rev "DEV")
+	)
 	(text "82p"
 		(exclude_from_sim no)
