File: TAPRX-888.kicad_pcb (KiCad board)
At the start: 6 copper layers, 83.5 x 99.4 mm, 225 parts, among them J1 CONN_SMA_JACK_EDGE_JLC_With_N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, J10 U.FL-R, J11 Conn_JTAG10-mini, J2 CONN_SMA_JACK_EDGE_JLC_With_N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, J3 CONN_SMA_JACK_EDGE_JLC_With_N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, J4 CONN_SMA_JACK_EDGE_JLC_With_N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, J5 USB-3.0, J6 Conn_01x03, J7 Conn_01x03, J8 Conn_01x03, J9 Conn_01x03, Q1 PMOS Si2343DS, Q2 MMBT3904, Q3 PMOS Si2343DS, U1 AP2114H-3.3TRG1, U10 XO-19.2MHZ, U11 CYUSB3014-BZXCT, U14 LP5907MFX-3.3, U16 TLV3501, U18 NC7SV157, U19 74LVC2G14, U2 AP2114H-3.3TRG1, U20 Si5351A, U21 NC7SV157, U22 SN65LVDS1, U3 AP2114H-3.3TRG1, U4 LP5907MFX-3.3, U5 UMW AMS1117-1.2, U6 AD8370, U7 TVS-SP3011, U8 LTC2208CUP#PBF, U9 MX25L3233FM2I, X1 TCXO-27M

Commit message: footprints: liberate from private TIS_Footprints library -> in-repo Library
Same TIS-liberation as the 3D models, footprint side. The board's 225 footprints
all claimed the private 'TIS_Footprints:' nickname, which isn't in the project
fp-lib-table (embedded geometry meant it still built, but the provenance pointed
at a library not in the repo).

- Extract the 2 footprints not yet in Library.pretty from the board's embedded
  copies (HamSCI-25mm; SMA_Jack_EdgeMount_JLC_With_Nut), stripped of instance
  data (position/uuid/nets, Reference -> REF**). Library.pretty now covers all 35.
- Re-point every board footprint lib-id 'TIS_Footprints:' -> 'Library:' (the
  in-repo library already defined in fp-lib-table as ${KIPRJMOD}/Library.pretty).
  Nickname rename only; embedded geometry unchanged.

Result: zero private-library references anywhere in the design. Every footprint
resolves from this repo's Library.pretty; every 3D model from KiCad's standard
library or this repo's 3d/.

Co-Authored-By: Claude Opus 4.8 <noreply@anthropic.com>
Claude-Session: https://claude.ai/code/session_01A68dcoDnizcNYhKvjGet5a
Parts:
- B1: footprint TIS_Footprints:BUTTON-4p5X4p5 -> Library:BUTTON-4p5X4p5
- C1, C10, C15, C16, C17, C18, C19, C2, C20, C21, C23, C24, C26, C27, C28, C3, C30, C31, C32, C34, C35, C36, C37, C38, C39, C40, C42, C43, C44, C46, C48, C49, C5, C50, C53, C54, C55, C56, C58, C59, C6, C61, C63, C64, C66, C67, C68, C69, C7, C70, C71, C72, C73, C74, C75, C76, C77, C8, C9: footprint TIS_Footprints:C_0603 -> Library:C_0603
- C11, C12, C13, C14, C22, C25, C29, C4, C41, C45, C47, C51, C52, C57, C60, C62, C65, C78, R1, R13, R14, R15, R16, R17, R18, R19, R2, R20, R21, R22, R23, R24, R25, R26, R27, R28, R29, R3, R30, R31, R32, R33, R34, R35, R36, R37, R38, R39, R4, R40, R41, R42, R43, R44, R45, R46, R47, R48, R49, R5, R50, R51, R52, R53, R54, R55, R56, R57, R58, R59, R6, R60, R61, R7, R8: footprint TIS_Footprints:PAD_0603 -> Library:PAD_0603
- C33: footprint TIS_Footprints:PAD_1206 -> Library:PAD_1206
- D1, D2: footprint TIS_Footprints:SOD-123 -> Library:SOD-123
- D3: footprint TIS_Footprints:LED_RGB_SIDE -> Library:LED_RGB_SIDE
- G***: footprint TIS_Footprints:HamSCI-25mm -> Library:HamSCI-25mm
- G***: footprint TIS_Footprints:TAPR 10mm -> Library:TAPR 10mm
- H1, H2, H3, H4: footprint TIS_Footprints:MountingHole_M2.5-PTH -> Library:MountingHole_M2.5-PTH
- J1, J2, J3, J4: footprint TIS_Footprints:SMA_Jack_EdgeMount_JLC_With_Nut -> Library:SMA_Jack_EdgeMount_JLC_With_Nut
- J10: footprint TIS_Footprints:HRS_U.FL-R-SMT(01) -> Library:HRS_U.FL-R-SMT(01)
- J11: footprint TIS_Footprints:CONN-JTAG10-mini -> Library:CONN-JTAG10-mini
- J5: footprint TIS_Footprints:USB-3.0 -> Library:USB-3.0
- J6, J7, J8, J9: footprint TIS_Footprints:Pin_Header_Straight_1x03_Pitch2.54mm -> Library:Pin_Header_Straight_1x03_Pitch2.54mm
- L1, L15, L16, L17, L3, L4, L5, L6, L7: footprint TIS_Footprints:0603 -> Library:0603
- L10, L11, L12, L13, L14, L8, L9: footprint TIS_Footprints:Murata2U -> Library:Murata2U
- L2: footprint TIS_Footprints:TIS-Logo -> Library:TIS-Logo
- Q1, Q2, Q3, U12, U13, U15, U17: footprint TIS_Footprints:SOT-23 -> Library:SOT-23
- R10, R11, R12, R9: footprint TIS_Footprints:4D02 -> Library:4D02
- TP1, TP10, TP11, TP12, TP13, TP14, TP15, TP16, TP17, TP18, TP19, TP2, TP3, TP4, TP5, TP6, TP7, TP8, TP9: footprint TIS_Footprints:TP -> Library:TP
- TP20, TP21: footprint TIS_Footprints:TP-Tiny -> Library:TP-Tiny
- U1, U2, U3, U5: footprint TIS_Footprints:SOT-223_THERMAL -> Library:SOT-223_THERMAL
- U10: footprint TIS_Footprints:SMD-2520 -> Library:SMD-2520
- U11: footprint TIS_Footprints:BGA-121 -> Library:BGA-121
- U14, U22, U4: footprint TIS_Footprints:SOT-23-5 -> Library:SOT-23-5
- U16: footprint TIS_Footprints:SOT-23-6 -> Library:SOT-23-6
- U18, U21: footprint TIS_Footprints:SC-70-6 -> Library:SC-70-6
- U19: footprint TIS_Footprints:SC-70-6_rot90 -> Library:SC-70-6_rot90
- U20: footprint TIS_Footprints:MSOP-10_W3mm -> Library:MSOP-10_W3mm
- U6: footprint TIS_Footprints:TSSOP-16-Thermal -> Library:TSSOP-16-Thermal
- U7: footprint TIS_Footprints:SP3011 -> Library:SP3011
- U8: footprint TIS_Footprints:QFN-64_EP_9.5x9.5_Pitch0.5mm -> Library:QFN-64_EP_9.5x9.5_Pitch0.5mm
- U9: footprint TIS_Footprints:SOIC-8-dual -> Library:SOIC-8-dual
- X1: footprint TIS_Footprints:TCXO-3225 -> Library:TCXO-3225
- Z1: footprint TIS_Footprints:SOD-323 -> Library:SOD-323

Commit message: footprints: put 0603 caps on C_0603; finish schematic TIS liberation
Fixes the one thing that made the board non-reproducible from the library: the
PAD_0603 footprint carried two 3D models (R_0603 for resistors, C_0603 for the
caps placed on it) via a board-level value override a single library footprint
can't express.

PAD_0603 and C_0603 are geometrically identical (same pads/silk), so:
- Reassign the 18 caps on PAD_0603 -> C_0603 (C4,C11-14,C22,C25,C29,C41,C45,C47,
  C51,C52,C57,C60,C62,C65,C78) in both the schematic (Footprint field) and the
  board. Zero copper change. Now PAD_0603 = resistors only (one model), C_0603 =
  caps only (one model); no per-instance model override remains.
- Finish the footprint liberation on the schematic side: re-point every
  schematic Footprint field TIS_Footprints: -> Library: (the board re-point had
  left the schematic mismatched).

Verified: no footprint type has >1 model; schematic Footprint fields == board
footprints for every part; zero TIS references anywhere; parens balanced.

Co-Authored-By: Claude Opus 4.8 <noreply@anthropic.com>
Claude-Session: https://claude.ai/code/session_01A68dcoDnizcNYhKvjGet5a
Parts:
- C11, C12, C13, C14, C22, C25, C29, C4, C41, C45, C47, C51, C52, C57, C60, C62, C65, C78: footprint Library:PAD_0603 -> Library:C_0603
Changed lines of the file:
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@@
 		)
 	)
-	(footprint "Library:PAD_0603"
+	(footprint "Library:C_0603"
 		(layer "F.Cu")
 		(at 138 71 90)
@@
 		)
 	)
-	(footprint "Library:PAD_0603"
+	(footprint "Library:C_0603"
 		(layer "F.Cu")
 		(at 170 96.125 180)
@@
 		)
 	)
-	(footprint "Library:PAD_0603"
+	(footprint "Library:C_0603"
 		(layer "F.Cu")
 		(at 149 73 180)
@@
 		)
 	)
-	(footprint "Library:PAD_0603"
+	(footprint "Library:C_0603"
 		(layer "F.Cu")
 		(at 140.2 116.1 180)
@@
 		)
 	)
-	(footprint "Library:PAD_0603"
+	(footprint "Library:C_0603"
 		(layer "F.Cu")
 		(at 149 77.5 180)
@@
 		)
 	)
-	(footprint "Library:PAD_0603"
+	(footprint "Library:C_0603"
 		(layer "F.Cu")
 		(at 149.25 82.95 180)
@@
 		)
 	)
-	(footprint "Library:PAD_0603"
+	(footprint "Library:C_0603"
 		(layer "F.Cu")
 		(at 108 72 -90)
@@
 		)
 	)
-	(footprint "Library:PAD_0603"
+	(footprint "Library:C_0603"
 		(layer "F.Cu")
 		(at 106 129 90)
@@
 		)
 	)
-	(footprint "Library:PAD_0603"
+	(footprint "Library:C_0603"
 		(layer "F.Cu")
 		(at 136 81)
@@
 		)
 	)
-	(footprint "Library:PAD_0603"
+	(footprint "Library:C_0603"
 		(layer "F.Cu")
 		(at 153 125)
@@
 		)
 	)
-	(footprint "Library:PAD_0603"
+	(footprint "Library:C_0603"
 		(layer "F.Cu")
 		(at 106 121 90)
@@
 		)
 	)
-	(footprint "Library:PAD_0603"
+	(footprint "Library:C_0603"
 		(layer "F.Cu")
 		(at 128 100 180)
@@
 		)
 	)
-	(footprint "Library:PAD_0603"
+	(footprint "Library:C_0603"
 		(layer "F.Cu")
 		(at 147.75 96.5 -90)
@@
 		)
 	)
-	(footprint "Library:PAD_0603"
+	(footprint "Library:C_0603"
 		(layer "F.Cu")
 		(at 170 90.125 180)
@@
 		)
 	)
-	(footprint "Library:PAD_0603"
+	(footprint "Library:C_0603"
 		(layer "F.Cu")
 		(at 141 90 180)
@@
 		)
 	)
-	(footprint "Library:PAD_0603"
+	(footprint "Library:C_0603"
 		(layer "F.Cu")
 		(at 128 125 180)
@@
 		)
 	)
-	(footprint "Library:PAD_0603"
+	(footprint "Library:C_0603"
 		(layer "F.Cu")
 		(at 140 109 180)
@@
 		)
 	)
-	(footprint "Library:PAD_0603"
+	(footprint "Library:C_0603"
 		(layer "F.Cu")
 		(at 118 57 90)
